Commit message: tried building ros2 gazebo bridge

File: ebot_description/models/ebot/ebot_description.xacro (robot description, xacro)
@@ -1,5 +1,4 @@
 <?xml version="1.0"?>
 <robot name="ebot" xmlns:xacro="http://www.ros.org/wiki/xacro">
-<xacro:include filename="$(find ebot_description)/models/ebot/ebot.gazebo" />
 <!-- macros for calculating inertia -->
 <xacro:property name="base_mass" value="46.034" />
@@ -929,27 +928,35 @@
     <dynamics damping="0.1" friction="10"/>
   </joint>
-  <ros2_control name="GazeboSystem" type="system">
-    <hardware>
-      <plugin>gazebo_ros2_control/GazeboSystem</plugin>
-    </hardware>
-    <joint name="linear_actuator_joint">
-      <command_interface name="effort">
-        <param name="min">-1000</param>
-        <param name="max">1000</param>
-      </command_interface>
-      <state_interface name="position">
-        <param name="initial_value">0.0</param>
-      </state_interface>
-      <state_interface name="velocity"/>
-      <state_interface name="effort"/>
-    </joint>
-  </ros2_control>
-<!--
   <gazebo>
-    <plugin filename="libgazebo_ros2_control.so" name="gazebo_ros2_control">
-      <robot_param>robot_description</robot_param>
-      <robot_param_node>ebot_RD</robot_param_node>
-      <parameters>$(find ebot_description)/config/controller.yaml</parameters>
+    <plugin
+        filename="libignition-gazebo-diff-drive-system.so"
+        name="ignition::gazebo::systems::DiffDrive">
+        <left_joint>FWLJ</left_joint>
+        <left_joint>RWLJ</left_joint>
+        <right_joint>FWRJ</right_joint>
+        <right_joint>RWRJ</right_joint>
+        <wheel_separation>1.2</wheel_separation>
+        <wheel_radius>0.4</wheel_radius>
+        <odom_publish_frequency>100.0</odom_publish_frequency>
+        <topic>cmd_vel</topic>
     </plugin>
-  </gazebo> -->
+      <plugin
+        filename="ignition-gazebo-joint-state-publisher-system"
+        name="ignition::gazebo::systems::JointStatePublisher">
+      </plugin>
+      <plugin
+        filename="ignition-gazebo-pose-publisher-system"
+        name="ignition::gazebo::systems::PosePublisher">
+        <publish_link_pose>true</publish_link_pose>
+        <use_pose_vector_msg>true</use_pose_vector_msg>
+        <static_publisher>true</static_publisher>
+        <static_update_frequency>1</static_update_frequency>
+      </plugin>
+      <plugin
+        filename="ignition-gazebo-odometry-publisher-system"
+        name="ignition::gazebo::systems::OdometryPublisher">
+        <odom_frame>ebot/odom</odom_frame>
+        <robot_base_frame>ebot</robot_base_frame>
+      </plugin>
+  </gazebo>
 </robot>
